Commit message: qu

File: ros2_ws/src/my_robot_description/urdf/my_robot.urdf.xacro (robot description, xacro)
@@ -118,5 +118,5 @@
     <parent link="base_link"/>
     <child link="imu_link"/>
-    <origin xyz="0.02 0 0.0459"
+    <origin xyz="0.02 0.12 0.0459"
             rpy="0 0 0"/>
 </joint>
@@ -168,5 +168,5 @@
     <parent link="base_cover_link"/>
     <child link="rplidar_link"/>
-    <origin xyz=".08 .07 .002"
+    <origin xyz=".12 .07 .002"
             rpy="0 0 0"/>
 </joint>

Commit message: repositioned bno055 in urdf

File: ros2_ws/src/my_robot_description/urdf/my_robot.urdf.xacro (robot description, xacro)
@@ -118,6 +118,6 @@
     <parent link="base_link"/>
     <child link="imu_link"/>
-    <origin xyz="0.02 0.12 0.0459"
-            rpy="0 0 0"/>
+    <origin xyz="0.055 0.125 0.0459"
+            rpy="0 -1.5708 0"/>
 </joint>
 <link name="camera_link">

Commit message: refactorede code a bit

File: ros2_ws/src/my_robot_description/urdf/my_robot.urdf.xacro (robot description, xacro)
@@ -178,290 +178,3 @@
             rpy="0 0 0"/>
 </joint>
-<!-- <link name="lidar_base_link">
-    <visual>
-        <geometry>
-            <mesh filename="package://my_robot_description/meshes/lidar_base.stl"
-                  scale="0.001 0.001 0.001"/>
-        </geometry>
-        <material name="gray">
-            <color rgba=".5 .5 .5 1"/>
-        </material>
-    </visual>
-    <collision>
-        <geometry>
-            <mesh filename="package://my_robot_description/meshes/lidar_base.stl"
-                  scale="0.001 0.001 0.001"/>
-        </geometry>
-    </collision>
-</link>
-<joint name="lidar_base_joint" type="fixed">
-    <parent link="base_link"/>
-    <child link="lidar_base_link"/>
-    <origin xyz=".05 .143 -0.0625"
-            rpy="1.5708 0 0"/>
-</joint>
-<link name="servo_link">
-    <visual>
-        <geometry>
-            <cylinder radius="0.02"
-                      length="0.02"/>
-        </geometry>
-        <material name="black">
-            <color rgba="0 1 0 1"/>
-        </material>
-    </visual>
-</link>
-<joint name="servo_rotation_joint" type="revolute">
-    <parent link="lidar_base_link"/>
-    <child link="servo_link"/>
-    <origin xyz=".04 .125 .0875"
-            rpy="-1.5708 3.14159 0"/>
-    <axis xyz="0 0 1"/>
-    <limit
-        lower=".52"
-        upper="2.62"
-        effort="2"
-        velocity="5"/>
-</joint>
-<link name="top_link">
-    <visual>
-        <geometry>
-            <mesh filename="package://my_robot_description/meshes/top.stl"
-                  scale="0.001 0.001 0.001"/>
-        </geometry>
-        <material name="gray">
-            <color rgba=".5 .5 .5 1"/>
-        </material>
-    </visual>
-</link>
-<joint name="top_joint" type="fixed">
-    <parent link="servo_link"/>
-    <child link="top_link"/>
-    <origin xyz="-.0375 .085 -.125"
-            rpy="1.5708 0 0"/>
-</joint>
-<link name="lidar_link">
-    <visual>
-        <geometry>
-            <box size="0.02125 0.035 0.012"/>
-        </geometry>
-        <origin xyz="0 0 0"/>
-        <material name="black">
-            <color rgba="0 0 0 1"/>
-        </material>
-    </visual>
-</link>
-<joint name="lidar_joint" type="fixed">
-    <parent link="top_link"/>
-    <child link="lidar_link"/>
-    <origin xyz=".04 .2 .09"
-            rpy="0 0 .785"/>
-</joint>
-<link name="shoulder_link">
-    <visual>
-        <geometry>
-            <mesh filename="package://my_robot_description/meshes/shoulder_small.stl"
-                  scale="0.001 0.001 0.001"/>
-        </geometry>
-        <material name="gray">
-            <color rgba="1 1 1 1"/>
-        </material>
-    </visual>
-    <collision>
-        <geometry>
-            <mesh filename="package://my_robot_description/meshes/shoulder_small.stl"
-                  scale="0.001 0.001 0.001"/>
-        </geometry>
-    </collision>
-</link>
-<joint name="shoulder_joint" type="fixed">
-    <parent link="top_link"/>
-    <child link="shoulder_link"/>
-    <origin xyz="0 0 0"
-            rpy="0 0 0"/>
-</joint>
-<link name="elbow_link">
-    <visual>
-        <geometry>
-            <mesh filename="package://my_robot_description/meshes/elbow_small.stl"
-                  scale="0.001 0.001 0.001"/>
-        </geometry>
-        <material name="gray">
-            <color rgba="1 1 1 1"/>
-        </material>
-    </visual>
-    <collision>
-        <geometry>
-            <mesh filename="package://my_robot_description/meshes/elbow_small.stl"
-                  scale="0.001 0.001 0.001"/>
-        </geometry>
-    </collision>
-</link>
-<joint name="elbow_joint" type="fixed">
-    <parent link="shoulder_link"/>
-    <child link="elbow_link"/>
-    <origin xyz="0 0 0"
-            rpy="0 0 0"/>
-</joint>
-<link name="base_gripper_link">
-    <visual>
-        <geometry>
-            <mesh filename="package://my_robot_description/meshes/base_gripper.stl"
-                  scale="0.001 0.001 0.001"/>
-        </geometry>
-        <material name="gray">
-            <color rgba="1 1 1 1"/>
-        </material>
-    </visual>
-    <collision>
-        <geometry>
-            <mesh filename="package://my_robot_description/meshes/base_gripper.stl"
-                  scale="0.001 0.001 0.001"/>
-        </geometry>
-    </collision>
-</link>
-<joint name="base_gripper_joint" type="fixed">
-    <parent link="elbow_link"/>
-    <child link="base_gripper_link"/>
-    <origin xyz="-.03 .155 .045"
-            rpy="0 0 0"/>
-</joint>
-<link name="gear1_link">
-    <visual>
-        <geometry>
-            <mesh filename="package://my_robot_description/meshes/gear1.stl"
-                  scale="0.001 0.001 0.001"/>
-        </geometry>
-        <material name="gray">
-            <color rgba="1 1 1 1"/>
-        </material>
-    </visual>
-    <collision>
-        <geometry>
-            <mesh filename="package://my_robot_description/meshes/gear1.stl"
-                  scale="0.001 0.001 0.001"/>
-        </geometry>
-    </collision>
-</link>
-<joint name="gear1_joint" type="fixed">
-    <parent link="base_gripper_link"/>
-    <child link="gear1_link"/>
-    <origin xyz="0 0 0"
-            rpy="0 0 0"/>
-</joint>
-<link name="gear2_link">
-    <visual>
-        <geometry>
-            <mesh filename="package://my_robot_description/meshes/gear2.stl"
-                  scale="0.001 0.001 0.001"/>
-        </geometry>
-        <material name="gray">
-            <color rgba="1 1 1 1"/>
-        </material>
-    </visual>
-    <collision>
-        <geometry>
-            <mesh filename="package://my_robot_description/meshes/gear2.stl"
-                  scale="0.001 0.001 0.001"/>
-        </geometry>
-    </collision>
-</link>
-<joint name="gear2_joint" type="fixed">
-    <parent link="base_gripper_link"/>
-    <child link="gear2_link"/>
-    <origin xyz="0 0 0"
-            rpy="0 0 0"/>
-</joint>
-<link name="bar1_link">
-    <visual>
-        <geometry>
-            <mesh filename="package://my_robot_description/meshes/bar1.stl"
-                  scale="0.001 0.001 0.001"/>
-        </geometry>
-        <material name="gray">
-            <color rgba="1 1 1 1"/>
-        </material>
-    </visual>
-    <collision>
-        <geometry>
-            <mesh filename="package://my_robot_description/meshes/bar1.stl"
-                  scale="0.001 0.001 0.001"/>
-        </geometry>
-    </collision>
-</link>
-<joint name="bar1_joint" type="fixed">
-    <parent link="base_gripper_link"/>
-    <child link="bar1_link"/>
-    <origin xyz="0 0 0"
-            rpy="0 0 0"/>
-</joint>
-<link name="bar2_link">
-    <visual>
-        <geometry>
-            <mesh filename="package://my_robot_description/meshes/bar2.stl"
-                  scale="0.001 0.001 0.001"/>
-        </geometry>
-        <material name="gray">
-            <color rgba="1 1 1 1"/>
-        </material>
-    </visual>
-    <collision>
-        <geometry>
-            <mesh filename="package://my_robot_description/meshes/bar2.stl"
-                  scale="0.001 0.001 0.001"/>
-        </geometry>
-    </collision>
-</link>
-<joint name="bar2_joint" type="fixed">
-    <parent link="base_gripper_link"/>
-    <child link="bar2_link"/>
-    <origin xyz="0 0 0"
-            rpy="0 0 0"/>
-</joint>
-<link name="gripper1_link">
-    <visual>
-        <geometry>
-            <mesh filename="package://my_robot_description/meshes/gripper1.stl"
-                  scale="0.001 0.001 0.001"/>
-        </geometry>
-        <material name="gray">
-            <color rgba="1 1 1 1"/>
-        </material>
-    </visual>
-    <collision>
-        <geometry>
-            <mesh filename="package://my_robot_description/meshes/gripper1.stl"
-                  scale="0.001 0.001 0.001"/>
-        </geometry>
-    </collision>
-</link>
-<joint name="gripper1_joint" type="fixed">
-    <parent link="base_gripper_link"/>
-    <child link="gripper1_link"/>
-    <origin xyz="0 0 0"
-            rpy="0 0 0"/>
-</joint>
-<link name="gripper2_link">
-    <visual>
-        <geometry>
-            <mesh filename="package://my_robot_description/meshes/gripper2.stl"
-                  scale="0.001 0.001 0.001"/>
-        </geometry>
-        <material name="gray">
-            <color rgba="1 1 1 1"/>
-        </material>
-    </visual>
-    <collision>
-        <geometry>
-            <mesh filename="package://my_robot_description/meshes/gripper2.stl"
-                  scale="0.001 0.001 0.001"/>
-        </geometry>
-    </collision>
-</link>
-<joint name="gripper2_joint" type="fixed">
-    <parent link="base_gripper_link"/>
-    <child link="gripper2_link"/>
-    <origin xyz="0 0 0"
-            rpy="0 0 0"/>
-</joint> -->
 </robot>
