Commit message: renamed my_robot to robot, started service conversion for arm_teleop

File: ros2_ws/src/arm_description/urdf/small_arm.urdf.xacro (robot description, xacro)
@@ -5,5 +5,5 @@
     <visual>
         <geometry>
-            <mesh filename="package://my_robot_description/meshes/lidar_base.stl"
+            <mesh filename="package://robot_description/meshes/lidar_base.stl"
                   scale="0.001 0.001 0.001"/>
         </geometry>
@@ -14,5 +14,5 @@
     <collision>
         <geometry>
-            <mesh filename="package://my_robot_description/meshes/lidar_base.stl"
+            <mesh filename="package://robot_description/meshes/lidar_base.stl"
                   scale="0.001 0.001 0.001"/>
         </geometry>
@@ -51,5 +51,5 @@
     <visual>
         <geometry>
-            <mesh filename="package://my_robot_description/meshes/top.stl"
+            <mesh filename="package://robot_description/meshes/top.stl"
                   scale="0.001 0.001 0.001"/>
         </geometry>
@@ -85,14 +85,14 @@
     <visual>
         <geometry>
-            <mesh filename="package://my_robot_description/meshes/shoulder_small.stl"
-                  scale="0.001 0.001 0.001"/>
-        </geometry>
-        <material name="gray">
-            <color rgba="1 1 1 1"/>
-        </material>
-    </visual>
-    <collision>
-        <geometry>
-            <mesh filename="package://my_robot_description/meshes/shoulder_small.stl"
+            <mesh filename="package://robot_description/meshes/shoulder_small.stl"
+                  scale="0.001 0.001 0.001"/>
+        </geometry>
+        <material name="gray">
+            <color rgba="1 1 1 1"/>
+        </material>
+    </visual>
+    <collision>
+        <geometry>
+            <mesh filename="package://robot_description/meshes/shoulder_small.stl"
                   scale="0.001 0.001 0.001"/>
         </geometry>
@@ -108,14 +108,14 @@
     <visual>
         <geometry>
-            <mesh filename="package://my_robot_description/meshes/elbow_small.stl"
-                  scale="0.001 0.001 0.001"/>
-        </geometry>
-        <material name="gray">
-            <color rgba="1 1 1 1"/>
-        </material>
-    </visual>
-    <collision>
-        <geometry>
-            <mesh filename="package://my_robot_description/meshes/elbow_small.stl"
+            <mesh filename="package://robot_description/meshes/elbow_small.stl"
+                  scale="0.001 0.001 0.001"/>
+        </geometry>
+        <material name="gray">
+            <color rgba="1 1 1 1"/>
+        </material>
+    </visual>
+    <collision>
+        <geometry>
+            <mesh filename="package://robot_description/meshes/elbow_small.stl"
                   scale="0.001 0.001 0.001"/>
         </geometry>
@@ -131,14 +131,14 @@
     <visual>
         <geometry>
-            <mesh filename="package://my_robot_description/meshes/base_gripper.stl"
-                  scale="0.001 0.001 0.001"/>
-        </geometry>
-        <material name="gray">
-            <color rgba="1 1 1 1"/>
-        </material>
-    </visual>
-    <collision>
-        <geometry>
-            <mesh filename="package://my_robot_description/meshes/base_gripper.stl"
+            <mesh filename="package://robot_description/meshes/base_gripper.stl"
+                  scale="0.001 0.001 0.001"/>
+        </geometry>
+        <material name="gray">
+            <color rgba="1 1 1 1"/>
+        </material>
+    </visual>
+    <collision>
+        <geometry>
+            <mesh filename="package://robot_description/meshes/base_gripper.stl"
                   scale="0.001 0.001 0.001"/>
         </geometry>
@@ -154,14 +154,14 @@
     <visual>
         <geometry>
-            <mesh filename="package://my_robot_description/meshes/gear1.stl"
-                  scale="0.001 0.001 0.001"/>
-        </geometry>
-        <material name="gray">
-            <color rgba="1 1 1 1"/>
-        </material>
-    </visual>
-    <collision>
-        <geometry>
-            <mesh filename="package://my_robot_description/meshes/gear1.stl"
+            <mesh filename="package://robot_description/meshes/gear1.stl"
+                  scale="0.001 0.001 0.001"/>
+        </geometry>
+        <material name="gray">
+            <color rgba="1 1 1 1"/>
+        </material>
+    </visual>
+    <collision>
+        <geometry>
+            <mesh filename="package://robot_description/meshes/gear1.stl"
                   scale="0.001 0.001 0.001"/>
         </geometry>
@@ -177,14 +177,14 @@
     <visual>
         <geometry>
-            <mesh filename="package://my_robot_description/meshes/gear2.stl"
-                  scale="0.001 0.001 0.001"/>
-        </geometry>
-        <material name="gray">
-            <color rgba="1 1 1 1"/>
-        </material>
-    </visual>
-    <collision>
-        <geometry>
-            <mesh filename="package://my_robot_description/meshes/gear2.stl"
+            <mesh filename="package://robot_description/meshes/gear2.stl"
+                  scale="0.001 0.001 0.001"/>
+        </geometry>
+        <material name="gray">
+            <color rgba="1 1 1 1"/>
+        </material>
+    </visual>
+    <collision>
+        <geometry>
+            <mesh filename="package://robot_description/meshes/gear2.stl"
                   scale="0.001 0.001 0.001"/>
         </geometry>
@@ -200,14 +200,14 @@
     <visual>
         <geometry>
-            <mesh filename="package://my_robot_description/meshes/bar1.stl"
-                  scale="0.001 0.001 0.001"/>
-        </geometry>
-        <material name="gray">
-            <color rgba="1 1 1 1"/>
-        </material>
-    </visual>
-    <collision>
-        <geometry>
-            <mesh filename="package://my_robot_description/meshes/bar1.stl"
+            <mesh filename="package://robot_description/meshes/bar1.stl"
+                  scale="0.001 0.001 0.001"/>
+        </geometry>
+        <material name="gray">
+            <color rgba="1 1 1 1"/>
+        </material>
+    </visual>
+    <collision>
+        <geometry>
+            <mesh filename="package://robot_description/meshes/bar1.stl"
                   scale="0.001 0.001 0.001"/>
         </geometry>
@@ -223,14 +223,14 @@
     <visual>
         <geometry>
-            <mesh filename="package://my_robot_description/meshes/bar2.stl"
-                  scale="0.001 0.001 0.001"/>
-        </geometry>
-        <material name="gray">
-            <color rgba="1 1 1 1"/>
-        </material>
-    </visual>
-    <collision>
-        <geometry>
-            <mesh filename="package://my_robot_description/meshes/bar2.stl"
+            <mesh filename="package://robot_description/meshes/bar2.stl"
+                  scale="0.001 0.001 0.001"/>
+        </geometry>
+        <material name="gray">
+            <color rgba="1 1 1 1"/>
+        </material>
+    </visual>
+    <collision>
+        <geometry>
+            <mesh filename="package://robot_description/meshes/bar2.stl"
                   scale="0.001 0.001 0.001"/>
         </geometry>
@@ -246,14 +246,14 @@
     <visual>
         <geometry>
-            <mesh filename="package://my_robot_description/meshes/gripper1.stl"
-                  scale="0.001 0.001 0.001"/>
-        </geometry>
-        <material name="gray">
-            <color rgba="1 1 1 1"/>
-        </material>
-    </visual>
-    <collision>
-        <geometry>
-            <mesh filename="package://my_robot_description/meshes/gripper1.stl"
+            <mesh filename="package://robot_description/meshes/gripper1.stl"
+                  scale="0.001 0.001 0.001"/>
+        </geometry>
+        <material name="gray">
+            <color rgba="1 1 1 1"/>
+        </material>
+    </visual>
+    <collision>
+        <geometry>
+            <mesh filename="package://robot_description/meshes/gripper1.stl"
                   scale="0.001 0.001 0.001"/>
         </geometry>
@@ -269,14 +269,14 @@
     <visual>
         <geometry>
-            <mesh filename="package://my_robot_description/meshes/gripper2.stl"
-                  scale="0.001 0.001 0.001"/>
-        </geometry>
-        <material name="gray">
-            <color rgba="1 1 1 1"/>
-        </material>
-    </visual>
-    <collision>
-        <geometry>
-            <mesh filename="package://my_robot_description/meshes/gripper2.stl"
+            <mesh filename="package://robot_description/meshes/gripper2.stl"
+                  scale="0.001 0.001 0.001"/>
+        </geometry>
+        <material name="gray">
+            <color rgba="1 1 1 1"/>
+        </material>
+    </visual>
+    <collision>
+        <geometry>
+            <mesh filename="package://robot_description/meshes/gripper2.stl"
                   scale="0.001 0.001 0.001"/>
         </geometry>

File: ros2_ws/src/robot_description/urdf/robot.urdf.xacro (robot description, xacro)
@@ -1,5 +1,5 @@
 <?xml version="1.0"?>
 <robot xmlns:xacro="http://www.ros.org/wiki/xacro"
-       name="my_robot">
+       name="robot">
 <xacro:property name="base_length" value="0.1500"/>
 <xacro:property name="base_width"  value="0.1250"/>
@@ -13,5 +13,5 @@
     <visual>
         <geometry>
-            <mesh filename="package://my_robot_description/meshes/base.stl"
+            <mesh filename="package://robot_description/meshes/base.stl"
                   scale="0.001 0.001 0.001"/>
         </geometry>
@@ -140,5 +140,5 @@
     <visual>
         <geometry>
-            <mesh filename="package://my_robot_description/meshes/base_cover.stl"
+            <mesh filename="package://robot_description/meshes/base_cover.stl"
                   scale="0.001 0.001 0.001"/>
         </geometry>
@@ -157,5 +157,5 @@
     <visual>
         <geometry>
-            <mesh filename="package://my_robot_description/meshes/rplidar.stl"
+            <mesh filename="package://robot_description/meshes/rplidar.stl"
                   scale="0.001 0.001 0.001"/>
         </geometry>
