Commit message: working on arm urdf

File: ros2_ws/src/arm_description/urdf/arm.urdf.xacro (robot description, xacro)
@@ -39,27 +39,4 @@
     <origin xyz="0 0 0" rpy="-1.5708 0 0"/>
 </joint>
-<!-- <link name="servo_link">
-    <visual>
-        <geometry>
-            <cylinder radius="0.02"
-                      length="0.02"/>
-        </geometry>
-        <material name="black">
-            <color rgba="0 0 0 1"/>
-        </material>
-    </visual>
-</link>
-<joint name="servo_rotation_joint" type="revolute">
-    <parent link="base_link"/>
-    <child link="servo_link"/>
-    <origin xyz="0 0 0"
-            rpy="0 0 0"/>
-    <axis xyz="0 1 0"/>
-    <limit
-        lower="-2.6"
-        upper="-.4"
-        effort="2"
-        velocity="5"/>
-</joint> -->
 <link name="central_axis_link">
     <visual>
@@ -68,5 +45,5 @@
                   scale="0.001 0.001 0.001"/>
         </geometry>
-        <material name="gray">
+        <material name="white">
             <color rgba="1 1 1 1"/>
         </material>
@@ -79,11 +56,17 @@
     </collision>
 </link>
-<joint name="central_axis_joint" type="fixed">
+<joint name="servo_rotation_joint" type="revolute">
     <parent link="base_link"/>
     <child link="central_axis_link"/>
     <origin xyz="0 0 0"
             rpy="0 0 0"/>
+    <axis xyz="0 0 1"/>
+    <limit
+        lower="-2.6"
+        upper="-.4"
+        effort="2"
+        velocity="5"/>
 </joint>
-<link name="shoulder_link">
+<!-- <link name="shoulder_link">
     <visual>
         <geometry>
@@ -176,4 +159,4 @@
     <origin xyz="-.21 .33 .048"
             rpy="1.5708 0 0"/>
-</joint>
+</joint> -->
 </robot>

Commit message: fixing arm kinematics

File: ros2_ws/src/arm_description/urdf/arm.urdf.xacro (robot description, xacro)
@@ -2,8 +2,10 @@
 <robot xmlns:xacro="http://www.ros.org/wiki/xacro"
        name="arm">
-<!-- <xacro:property name="base_length" value="0.1500"/> -->
 <link name="world"/>
 <link name="base_link">
     <visual>
+        <origin
+            xyz="-0.04035 0.09275 -0.10300"
+            rpy="1.5708 0 0"/>
         <geometry>
             <mesh filename="package://arm_description/meshes/base.stl"
@@ -15,5 +17,7 @@
     </visual>
     <collision>
-     <origin xyz="0 0 0" rpy="0 0 0"/>
+        <origin
+            xyz="-0.04035 0.09275 -0.10300"
+            rpy="1.5708 0 0"/>
         <geometry>
             <mesh filename="package://arm_description/meshes/base.stl"
@@ -36,9 +40,11 @@
     <parent link="world"/>
     <child link="base_link"/>
-    <!-- Change these values to move or rotate the entire robot -->
-    <origin xyz="0 0 0" rpy="-1.5708 0 0"/>
+    <origin xyz="0 0 0" rpy="0 0 0"/>
 </joint>
 <link name="central_axis_link">
     <visual>
+        <origin
+            xyz="-0.04035 0.09275 -0.10300"
+            rpy="1.5708 0 0"/>
         <geometry>
             <mesh filename="package://arm_description/meshes/central_axis.stl"
@@ -50,4 +56,7 @@
     </visual>
     <collision>
+        <origin
+            xyz="-0.04035 0.09275 -0.10300"
+            rpy="1.5708 0 0"/>
         <geometry>
             <mesh filename="package://arm_description/meshes/central_axis.stl"
@@ -68,6 +77,9 @@
         velocity="5"/>
 </joint>
-<!-- <link name="shoulder_link">
-    <visual>
+<link name="shoulder_link">
+    <visual>
+         <origin
+            xyz="-0.02885 0.09287 -0.16145"
+            rpy="1.5708 0 0"/>
         <geometry>
             <mesh filename="package://arm_description/meshes/shoulder.stl"
@@ -79,4 +91,7 @@
     </visual>
     <collision>
+         <origin
+            xyz="-0.02885 0.09287 -0.16145"
+            rpy="1.5708 0 0"/>
         <geometry>
             <mesh filename="package://arm_description/meshes/shoulder.stl"
@@ -85,12 +100,21 @@
     </collision>
 </link>
-<joint name="shoulder_joint" type="fixed">
+<joint name="shoulder_joint" type="revolute">
     <parent link="central_axis_link"/>
     <child link="shoulder_link"/>
-    <origin xyz="0 0 0"
-            rpy="0 0 0"/>
+    <origin xyz="-0.01150 0 0.05845"
+            rpy="0 0 0"/>
+    <axis xyz="0 1 0"/>
+    <limit
+        lower="-2.6"
+        upper="-.4"
+        effort="2"
+        velocity="5"/>
 </joint>
 <link name="elbow_link">
     <visual>
+        <origin
+            xyz="0 0 0"
+            rpy="1.5708 0 0"/>
         <geometry>
             <mesh filename="package://arm_description/meshes/elbow.stl"
@@ -102,4 +126,7 @@
     </visual>
     <collision>
+        <origin
+            xyz="0 0 0"
+            rpy="1.5708 0 0"/>
         <geometry>
             <mesh filename="package://arm_description/meshes/elbow.stl"
@@ -113,7 +140,16 @@
     <origin xyz="0 0 0"
             rpy="0 0 0"/>
-</joint>
-<link name="wrist_link">
-    <visual>
+    <axis xyz="0 1 0"/>
+    <limit
+        lower="-2.6"
+        upper="-.4"
+        effort="2"
+        velocity="5"/>
+</joint>
+<!-- <link name="wrist_link">
+    <visual>
+        <origin
+            xyz="-0.04035 0.09275 -0.10300"
+            rpy="1.5708 0 0"/>
         <geometry>
             <mesh filename="package://arm_description/meshes/wrist.stl"
@@ -125,4 +161,7 @@
     </visual>
     <collision>
+        <origin
+            xyz="-0.04035 0.09275 -0.10300"
+            rpy="1.5708 0 0"/>
         <geometry>
             <mesh filename="package://arm_description/meshes/wrist.stl"
@@ -136,7 +175,16 @@
     <origin xyz="0 0 0"
             rpy="0 0 0"/>
+    <axis xyz="0 0 1"/>
+    <limit
+        lower="-2.6"
+        upper="-.4"
+        effort="2"
+        velocity="5"/>
 </joint>
 <link name="gripper_link">
     <visual>
+        <origin
+            xyz="-0.04035 0.09275 -0.10300"
+            rpy="1.5708 0 0"/>
         <geometry>
             <mesh filename="package://arm_description/meshes/gripper.stl"
@@ -148,4 +196,7 @@
     </visual>
     <collision>
+        <origin
+            xyz="-0.04035 0.09275 -0.10300"
+            rpy="1.5708 0 0"/>
         <geometry>
             <mesh filename="package://arm_description/meshes/gripper.stl"
@@ -159,4 +210,10 @@
     <origin xyz="-.21 .33 .048"
             rpy="1.5708 0 0"/>
+    <axis xyz="0 0 1"/>
+    <limit
+        lower="-2.6"
+        upper="-.4"
+        effort="2"
+        velocity="5"/>
 </joint> -->
 </robot>

Commit message: solving for elbow link and joint

File: ros2_ws/src/arm_description/urdf/arm.urdf.xacro (robot description, xacro)
@@ -115,5 +115,5 @@
     <visual>
         <origin
-            xyz="0 0 0"
+            xyz="-0.03110 0.09267 -0.28350"
             rpy="1.5708 0 0"/>
         <geometry>
@@ -127,5 +127,5 @@
     <collision>
         <origin
-            xyz="0 0 0"
+            xyz="-0.03110 0.09267 -0.28350"
             rpy="1.5708 0 0"/>
         <geometry>
@@ -138,5 +138,5 @@
     <parent link="shoulder_link"/>
     <child link="elbow_link"/>
-    <origin xyz="0 0 0"
+    <origin xyz="0.00225 0 0.12205"
             rpy="0 0 0"/>
     <axis xyz="0 1 0"/>

Commit message: fixed wrist link and joint

File: ros2_ws/src/arm_description/urdf/arm.urdf.xacro (robot description, xacro)
@@ -107,6 +107,6 @@
     <axis xyz="0 1 0"/>
     <limit
-        lower="-2.6"
-        upper="-.4"
+        lower="-2"
+        upper="1"
         effort="2"
         velocity="5"/>
@@ -135,5 +135,5 @@
     </collision>
 </link>
-<joint name="elbow_joint" type="fixed">
+<joint name="elbow_joint" type="revolute">
     <parent link="shoulder_link"/>
     <child link="elbow_link"/>
@@ -142,4 +142,39 @@
     <axis xyz="0 1 0"/>
     <limit
+        lower="-.4"
+        upper="2.6"
+        effort="2"
+        velocity="5"/>
+</joint>
+<link name="wrist_link">
+    <visual>
+        <origin
+            xyz="0.059395 0.10537 -0.302995"
+            rpy="1.5708 0 0"/>
+        <geometry>
+            <mesh filename="package://arm_description/meshes/wrist.stl"
+                  scale="0.001 0.001 0.001"/>
+        </geometry>
+        <material name="gray">
+            <color rgba="1 1 1 1"/>
+        </material>
+    </visual>
+    <collision>
+        <origin
+            xyz="0.059395 0.10537 -0.302995"
+            rpy="1.5708 0 0"/>
+        <geometry>
+            <mesh filename="package://arm_description/meshes/wrist.stl"
+                  scale="0.001 0.001 0.001"/>
+        </geometry>
+    </collision>
+</link>
+<joint name="wrist_joint" type="revolute">
+    <parent link="elbow_link"/>
+    <child link="wrist_link"/>
+    <origin xyz="-0.090495 -0.01270 0.019495"
+            rpy="0 0 0"/>
+    <axis xyz="1 0 0"/>
+    <limit
         lower="-2.6"
         upper="-.4"
@@ -147,39 +182,4 @@
         velocity="5"/>
 </joint>
-<!-- <link name="wrist_link">
-    <visual>
-        <origin
-            xyz="-0.04035 0.09275 -0.10300"
-            rpy="1.5708 0 0"/>
-        <geometry>
-            <mesh filename="package://arm_description/meshes/wrist.stl"
-                  scale="0.001 0.001 0.001"/>
-        </geometry>
-        <material name="gray">
-            <color rgba="1 1 1 1"/>
-        </material>
-    </visual>
-    <collision>
-        <origin
-            xyz="-0.04035 0.09275 -0.10300"
-            rpy="1.5708 0 0"/>
-        <geometry>
-            <mesh filename="package://arm_description/meshes/wrist.stl"
-                  scale="0.001 0.001 0.001"/>
-        </geometry>
-    </collision>
-</link>
-<joint name="wrist_joint" type="fixed">
-    <parent link="elbow_link"/>
-    <child link="wrist_link"/>
-    <origin xyz="0 0 0"
-            rpy="0 0 0"/>
-    <axis xyz="0 0 1"/>
-    <limit
-        lower="-2.6"
-        upper="-.4"
-        effort="2"
-        velocity="5"/>
-</joint>
 <link name="gripper_link">
     <visual>
@@ -205,5 +205,5 @@
     </collision>
 </link>
-<joint name="gripper_joint" type="fixed">
+<joint name="gripper_joint" type="revolute">
     <parent link="wrist_link"/>
     <child link="gripper_link"/>
@@ -216,4 +216,4 @@
         effort="2"
         velocity="5"/>
-</joint> -->
+</joint>
 </robot>

Commit message: added gripper forward kinematicd

File: ros2_ws/src/arm_description/urdf/arm.urdf.xacro (robot description, xacro)
@@ -86,5 +86,5 @@
                   scale="0.001 0.001 0.001"/>
         </geometry>
-        <material name="gray">
+        <material name="white">
             <color rgba="1 1 1 1"/>
         </material>
@@ -121,5 +121,5 @@
                   scale="0.001 0.001 0.001"/>
         </geometry>
-        <material name="gray">
+        <material name="white">
             <color rgba="1 1 1 1"/>
         </material>
@@ -156,6 +156,6 @@
                   scale="0.001 0.001 0.001"/>
         </geometry>
-        <material name="gray">
-            <color rgba="1 1 1 1"/>
+        <material name="black">
+            <color rgba="0 0 0 1"/>
         </material>
     </visual>
@@ -185,5 +185,5 @@
     <visual>
         <origin
-            xyz="-0.04035 0.09275 -0.10300"
+            xyz="-0.11823 0.01750 -0.03923"
             rpy="1.5708 0 0"/>
         <geometry>
@@ -191,11 +191,11 @@
                   scale="0.001 0.001 0.001"/>
         </geometry>
-        <material name="gray">
-            <color rgba="1 1 1 1"/>
-        </material>
-    </visual>
-    <collision>
-        <origin
-            xyz="-0.04035 0.09275 -0.10300"
+        <material name="white">
+            <color rgba="1 1 1 1"/>
+        </material>
+    </visual>
+    <collision>
+        <origin
+            xyz="-0.11823 0.01750 -0.03923"
             rpy="1.5708 0 0"/>
         <geometry>
@@ -208,10 +208,10 @@
     <parent link="wrist_link"/>
     <child link="gripper_link"/>
-    <origin xyz="-.21 .33 .048"
+    <origin xyz="-0.026525 0.013365 0.005365"
             rpy="1.5708 0 0"/>
     <axis xyz="0 0 1"/>
     <limit
-        lower="-2.6"
-        upper="-.4"
+        lower="-2"
+        upper="1"
         effort="2"
         velocity="5"/>

Commit message: transitioning from joint_state-publisher_gui to actual robot arm

File: ros2_ws/src/arm_description/urdf/arm.urdf.xacro (robot description, xacro)
@@ -65,5 +65,5 @@
     </collision>
 </link>
-<joint name="servo_rotation_joint" type="revolute">
+<joint name="base_joint" type="revolute">
     <parent link="base_link"/>
     <child link="central_axis_link"/>
@@ -182,5 +182,5 @@
         velocity="5"/>
 </joint>
-<link name="gripper_link">
+<link name="gripper1_link">
     <visual>
         <origin
@@ -205,7 +205,7 @@
     </collision>
 </link>
-<joint name="gripper_joint" type="revolute">
+<joint name="gripper1_joint" type="revolute">
     <parent link="wrist_link"/>
-    <child link="gripper_link"/>
+    <child link="gripper1_link"/>
     <origin xyz="-0.026525 0.013365 0.005365"
             rpy="1.5708 0 0"/>
@@ -217,3 +217,15 @@
         velocity="5"/>
 </joint>
+<link name="gripper2_link"/>
+<joint name="gripper2_joint" type="revolute">
+    <parent link="gripper1_link"/>
+    <child link="gripper2_link"/>
+    <origin xyz="-0.012505 0.017492 -0.027285"
+            rpy="0 0 0"/>
+    <axis xyz="0 0 1"/>
+    <limit lower="0"
+           upper="1.57"
+           effort="2"
+           velocity="5"/>
+</joint>
 </robot>

Commit message: test jacobian

File: ros2_ws/src/arm_description/urdf/arm.urdf.xacro (robot description, xacro)
@@ -223,5 +223,5 @@
     <origin xyz="-0.012505 0.017492 -0.027285"
             rpy="0 0 0"/>
-    <axis xyz="0 0 1"/>
+    <axis xyz="1 0 0"/>
     <limit lower="0"
            upper="1.57"

Commit message: one iteration of numericla inverse kienmatics

File: ros2_ws/src/arm_description/urdf/arm.urdf.xacro (robot description, xacro)
@@ -65,5 +65,5 @@
     </collision>
 </link>
-<joint name="base_joint" type="revolute">
+<joint name="central_axis_joint" type="revolute">
     <parent link="base_link"/>
     <child link="central_axis_link"/>

Commit message: completed and tested forward and inverse kinematics in rviz, now just need to match the angles for actual robot arm to how they move in rviz

File: ros2_ws/src/arm_description/urdf/arm.urdf.xacro (robot description, xacro)
@@ -229,3 +229,9 @@
            velocity="5"/>
 </joint>
+<link name="tool_link"/>
+<joint name="tool_joint" type="fixed">
+    <parent link="gripper2_link"/>
+    <child link="tool_link"/>
+    <origin xyz="-0.05 0 0" rpy="0 0 0"/>
+</joint>
 </robot>
